File: pcb/matrix.kicad_sch (KiCad schematic)
At the start: 176 parts

Commit message: Schematic completed
Parts:
- D1: footprint footprints:D_0603_1608Metric -> diodes:D-0603-1608
- D10, D11, D12, D13, D14, D15, D16, D17, D18, D19, D2, D20, D21, D22, D23, D24, D25, D26, D27, D28, D29, D3, D30, D31, D32, D33, D34, D35, D36, D37, D38, D39, D4, D40, D41, D42, D43, D44, D45, D46, D47, D48, D49, D5, D50, D51, D52, D53, D54, D55, D56, D57, D58, D59, D6, D60, D61, D62, D63, D64, D65, D66, D67, D68, D69, D7, D70, D71, D72, D73, D74, D75, D76, D77, D78, D79, D8, D80, D81, D82, D83, D84, D85, D86, D87, D88, D9: value D_Small -> (none); footprint footprints:D_0603_1608Metric -> diodes:D-0603-1608
- MX1: footprint footprints:SW-Kailh-Hotswap-MX-1.00u -> switches:SW-Kailh-Hotswap-MX-1.00u; symbol MX_Switch:MX-NoLED -> MX-Switch:MX-NoLED
- MX10: value F9 -> (none); footprint footprints:SW-Kailh-Hotswap-MX-1.00u -> switches:SW-Kailh-Hotswap-MX-1.00u; symbol MX_Switch:MX-NoLED -> MX-Switch:MX-NoLED
- MX11: value F10 -> (none); footprint footprints:SW-Kailh-Hotswap-MX-1.00u -> switches:SW-Kailh-Hotswap-MX-1.00u; symbol MX_Switch:MX-NoLED -> MX-Switch:MX-NoLED
- MX12: value F11 -> (none); footprint footprints:SW-Kailh-Hotswap-MX-1.00u -> switches:SW-Kailh-Hotswap-MX-1.00u; symbol MX_Switch:MX-NoLED -> MX-Switch:MX-NoLED
- MX13: value F12 -> (none); footprint footprints:SW-Kailh-Hotswap-MX-1.00u -> switches:SW-Kailh-Hotswap-MX-1.00u; symbol MX_Switch:MX-NoLED -> MX-Switch:MX-NoLED
- MX14: value F13 -> (none); footprint footprints:SW-Kailh-Hotswap-MX-1.00u -> switches:SW-Kailh-Hotswap-MX-1.00u; symbol MX_Switch:MX-NoLED -> MX-Switch:MX-NoLED
- MX15: value PrtSc -> (none); footprint footprints:SW-Kailh-Hotswap-MX-1.00u -> switches:SW-Kailh-Hotswap-MX-1.00u; symbol MX_Switch:MX-NoLED -> MX-Switch:MX-NoLED
- MX16: value ScrLck -> (none); footprint footprints:SW-Kailh-Hotswap-MX-1.00u -> switches:SW-Kailh-Hotswap-MX-1.00u; symbol MX_Switch:MX-NoLED -> MX-Switch:MX-NoLED
- MX17: value Pause -> (none); footprint footprints:SW-Kailh-Hotswap-MX-1.00u -> switches:SW-Kailh-Hotswap-MX-1.00u; symbol MX_Switch:MX-NoLED -> MX-Switch:MX-NoLED
- MX18: value ~ -> (none); footprint footprints:SW-Kailh-Hotswap-MX-1.00u -> switches:SW-Kailh-Hotswap-MX-1.00u; symbol MX_Switch:MX-NoLED -> MX-Switch:MX-NoLED
- MX19: value 1 -> (none); footprint footprints:SW-Kailh-Hotswap-MX-1.00u -> switches:SW-Kailh-Hotswap-MX-1.00u; symbol MX_Switch:MX-NoLED -> MX-Switch:MX-NoLED
- MX2: value F1 -> (none); footprint footprints:SW-Kailh-Hotswap-MX-1.00u -> switches:SW-Kailh-Hotswap-MX-1.00u; symbol MX_Switch:MX-NoLED -> MX-Switch:MX-NoLED
- MX20: value 2 -> (none); footprint footprints:SW-Kailh-Hotswap-MX-1.00u -> switches:SW-Kailh-Hotswap-MX-1.00u; symbol MX_Switch:MX-NoLED -> MX-Switch:MX-NoLED
- MX21: value 3 -> (none); footprint footprints:SW-Kailh-Hotswap-MX-1.00u -> switches:SW-Kailh-Hotswap-MX-1.00u; symbol MX_Switch:MX-NoLED -> MX-Switch:MX-NoLED
- MX22: value 4 -> (none); footprint footprints:SW-Kailh-Hotswap-MX-1.00u -> switches:SW-Kailh-Hotswap-MX-1.00u; symbol MX_Switch:MX-NoLED -> MX-Switch:MX-NoLED
- MX23: value 5 -> (none); footprint footprints:SW-Kailh-Hotswap-MX-1.00u -> switches:SW-Kailh-Hotswap-MX-1.00u; symbol MX_Switch:MX-NoLED -> MX-Switch:MX-NoLED
- MX24: value 6 -> (none); footprint footprints:SW-Kailh-Hotswap-MX-1.00u -> switches:SW-Kailh-Hotswap-MX-1.00u; symbol MX_Switch:MX-NoLED -> MX-Switch:MX-NoLED
- MX25: value 7 -> (none); footprint footprints:SW-Kailh-Hotswap-MX-1.00u -> switches:SW-Kailh-Hotswap-MX-1.00u; symbol MX_Switch:MX-NoLED -> MX-Switch:MX-NoLED
- MX26: value 8 -> (none); footprint footprints:SW-Kailh-Hotswap-MX-1.00u -> switches:SW-Kailh-Hotswap-MX-1.00u; symbol MX_Switch:MX-NoLED -> MX-Switch:MX-NoLED
- MX27: value 9 -> (none); footprint footprints:SW-Kailh-Hotswap-MX-1.00u -> switches:SW-Kailh-Hotswap-MX-1.00u; symbol MX_Switch:MX-NoLED -> MX-Switch:MX-NoLED
- MX28: value 0 -> (none); footprint footprints:SW-Kailh-Hotswap-MX-1.00u -> switches:SW-Kailh-Hotswap-MX-1.00u; symbol MX_Switch:MX-NoLED -> MX-Switch:MX-NoLED
- MX29: value - -> (none); footprint footprints:SW-Kailh-Hotswap-MX-1.00u -> switches:SW-Kailh-Hotswap-MX-1.00u; symbol MX_Switch:MX-NoLED -> MX-Switch:MX-NoLED
- MX3: value F2 -> (none); footprint footprints:SW-Kailh-Hotswap-MX-1.00u -> switches:SW-Kailh-Hotswap-MX-1.00u; symbol MX_Switch:MX-NoLED -> MX-Switch:MX-NoLED
- MX30: value + -> (none); footprint footprints:SW-Kailh-Hotswap-MX-1.00u -> switches:SW-Kailh-Hotswap-MX-1.00u; symbol MX_Switch:MX-NoLED -> MX-Switch:MX-NoLED
- MX31: value Bck -> (none); footprint footprints:SW-Kailh-Hotswap-MX-2.00u -> switches:SW-Kailh-Hotswap-MX-2.00u; symbol MX_Switch:MX-NoLED -> MX-Switch:MX-NoLED
- MX32: value Insert -> (none); footprint footprints:SW-Kailh-Hotswap-MX-1.00u -> switches:SW-Kailh-Hotswap-MX-1.00u; symbol MX_Switch:MX-NoLED -> MX-Switch:MX-NoLED
- MX33: value Home -> (none); footprint footprints:SW-Kailh-Hotswap-MX-1.00u -> switches:SW-Kailh-Hotswap-MX-1.00u; symbol MX_Switch:MX-NoLED -> MX-Switch:MX-NoLED
- MX34: value PgUp -> (none); footprint footprints:SW-Kailh-Hotswap-MX-1.00u -> switches:SW-Kailh-Hotswap-MX-1.00u; symbol MX_Switch:MX-NoLED -> MX-Switch:MX-NoLED
- MX35: value Tab -> (none); footprint footprints:SW-Kailh-Hotswap-MX-1.50u -> switches:SW-Kailh-Hotswap-MX-1.50u; symbol MX_Switch:MX-NoLED -> MX-Switch:MX-NoLED
- MX36: value Q -> (none); footprint footprints:SW-Kailh-Hotswap-MX-1.00u -> switches:SW-Kailh-Hotswap-MX-1.00u; symbol MX_Switch:MX-NoLED -> MX-Switch:MX-NoLED
- MX37: value W -> (none); footprint footprints:SW-Kailh-Hotswap-MX-1.00u -> switches:SW-Kailh-Hotswap-MX-1.00u; symbol MX_Switch:MX-NoLED -> MX-Switch:MX-NoLED
- MX38: value E -> (none); footprint footprints:SW-Kailh-Hotswap-MX-1.00u -> switches:SW-Kailh-Hotswap-MX-1.00u; symbol MX_Switch:MX-NoLED -> MX-Switch:MX-NoLED
- MX39: value R -> (none); footprint footprints:SW-Kailh-Hotswap-MX-1.00u -> switches:SW-Kailh-Hotswap-MX-1.00u; symbol MX_Switch:MX-NoLED -> MX-Switch:MX-NoLED
- MX4: value F3 -> (none); footprint footprints:SW-Kailh-Hotswap-MX-1.00u -> switches:SW-Kailh-Hotswap-MX-1.00u; symbol MX_Switch:MX-NoLED -> MX-Switch:MX-NoLED
- MX40: value T -> (none); footprint footprints:SW-Kailh-Hotswap-MX-1.00u -> switches:SW-Kailh-Hotswap-MX-1.00u; symbol MX_Switch:MX-NoLED -> MX-Switch:MX-NoLED
- MX41: value Y -> (none); footprint footprints:SW-Kailh-Hotswap-MX-1.00u -> switches:SW-Kailh-Hotswap-MX-1.00u; symbol MX_Switch:MX-NoLED -> MX-Switch:MX-NoLED
- MX42: value U -> (none); footprint footprints:SW-Kailh-Hotswap-MX-1.00u -> switches:SW-Kailh-Hotswap-MX-1.00u; symbol MX_Switch:MX-NoLED -> MX-Switch:MX-NoLED
- MX43: value I -> (none); footprint footprints:SW-Kailh-Hotswap-MX-1.00u -> switches:SW-Kailh-Hotswap-MX-1.00u; symbol MX_Switch:MX-NoLED -> MX-Switch:MX-NoLED
- MX44: value O -> (none); footprint footprints:SW-Kailh-Hotswap-MX-1.00u -> switches:SW-Kailh-Hotswap-MX-1.00u; symbol MX_Switch:MX-NoLED -> MX-Switch:MX-NoLED
- MX45: value P -> (none); footprint footprints:SW-Kailh-Hotswap-MX-1.00u -> switches:SW-Kailh-Hotswap-MX-1.00u; symbol MX_Switch:MX-NoLED -> MX-Switch:MX-NoLED
- MX46: value [ -> (none); footprint footprints:SW-Kailh-Hotswap-MX-1.00u -> switches:SW-Kailh-Hotswap-MX-1.00u; symbol MX_Switch:MX-NoLED -> MX-Switch:MX-NoLED
- MX47: value ] -> (none); footprint footprints:SW-Kailh-Hotswap-MX-1.00u -> switches:SW-Kailh-Hotswap-MX-1.00u; symbol MX_Switch:MX-NoLED -> MX-Switch:MX-NoLED
- MX48: value \ -> (none); footprint footprints:SW-Kailh-Hotswap-MX-1.50u -> switches:SW-Kailh-Hotswap-MX-1.00u; symbol MX_Switch:MX-NoLED -> MX-Switch:MX-NoLED
- MX49: value Delete -> (none); footprint footprints:SW-Kailh-Hotswap-MX-1.00u -> switches:SW-Kailh-Hotswap-MX-1.00u; symbol MX_Switch:MX-NoLED -> MX-Switch:MX-NoLED
- MX5: value F4 -> (none); footprint footprints:SW-Kailh-Hotswap-MX-1.00u -> switches:SW-Kailh-Hotswap-MX-1.00u; symbol MX_Switch:MX-NoLED -> MX-Switch:MX-NoLED
- MX50: value End -> (none); footprint footprints:SW-Kailh-Hotswap-MX-1.00u -> switches:SW-Kailh-Hotswap-MX-1.00u; symbol MX_Switch:MX-NoLED -> MX-Switch:MX-NoLED
- MX51: value PgDn -> (none); footprint footprints:SW-Kailh-Hotswap-MX-1.00u -> switches:SW-Kailh-Hotswap-MX-1.00u; symbol MX_Switch:MX-NoLED -> MX-Switch:MX-NoLED
- MX52: value Caps -> (none); footprint footprints:SW-Kailh-Hotswap-MX-1.75u -> switches:SW-Kailh-Hotswap-MX-1.75u; symbol MX_Switch:MX-NoLED -> MX-Switch:MX-NoLED
- MX53: value A -> (none); footprint footprints:SW-Kailh-Hotswap-MX-1.00u -> switches:SW-Kailh-Hotswap-MX-1.00u; symbol MX_Switch:MX-NoLED -> MX-Switch:MX-NoLED
- MX54: value S -> (none); footprint footprints:SW-Kailh-Hotswap-MX-1.00u -> switches:SW-Kailh-Hotswap-MX-1.00u; symbol MX_Switch:MX-NoLED -> MX-Switch:MX-NoLED
- MX55: value D -> (none); footprint footprints:SW-Kailh-Hotswap-MX-1.00u -> switches:SW-Kailh-Hotswap-MX-1.00u; symbol MX_Switch:MX-NoLED -> MX-Switch:MX-NoLED
- MX56: value F -> (none); footprint footprints:SW-Kailh-Hotswap-MX-1.00u -> switches:SW-Kailh-Hotswap-MX-1.00u; symbol MX_Switch:MX-NoLED -> MX-Switch:MX-NoLED
- MX57: value G -> (none); footprint footprints:SW-Kailh-Hotswap-MX-1.00u -> switches:SW-Kailh-Hotswap-MX-1.00u; symbol MX_Switch:MX-NoLED -> MX-Switch:MX-NoLED
- MX58: value H -> (none); footprint footprints:SW-Kailh-Hotswap-MX-1.00u -> switches:SW-Kailh-Hotswap-MX-1.00u; symbol MX_Switch:MX-NoLED -> MX-Switch:MX-NoLED
- MX59: value J -> (none); footprint footprints:SW-Kailh-Hotswap-MX-1.00u -> switches:SW-Kailh-Hotswap-MX-1.00u; symbol MX_Switch:MX-NoLED -> MX-Switch:MX-NoLED
- MX6: value F5 -> (none); footprint footprints:SW-Kailh-Hotswap-MX-1.00u -> switches:SW-Kailh-Hotswap-MX-1.00u; symbol MX_Switch:MX-NoLED -> MX-Switch:MX-NoLED
- MX60: value K -> (none); footprint footprints:SW-Kailh-Hotswap-MX-1.00u -> switches:SW-Kailh-Hotswap-MX-1.00u; symbol MX_Switch:MX-NoLED -> MX-Switch:MX-NoLED
- MX61: value L -> (none); footprint footprints:SW-Kailh-Hotswap-MX-1.00u -> switches:SW-Kailh-Hotswap-MX-1.00u; symbol MX_Switch:MX-NoLED -> MX-Switch:MX-NoLED
- MX62: value ; -> (none); footprint footprints:SW-Kailh-Hotswap-MX-1.00u -> switches:SW-Kailh-Hotswap-MX-1.00u; symbol MX_Switch:MX-NoLED -> MX-Switch:MX-NoLED
- MX63: value ' -> (none); footprint footprints:SW-Kailh-Hotswap-MX-1.00u -> switches:SW-Kailh-Hotswap-MX-1.00u; symbol MX_Switch:MX-NoLED -> MX-Switch:MX-NoLED
- MX64: value Enter -> (none); footprint footprints:SW-Kailh-Hotswap-MX-2.25u -> switches:SW-Kailh-Hotswap-MX-2.25u; symbol MX_Switch:MX-NoLED -> MX-Switch:MX-NoLED
- MX65: value LShift -> (none); footprint footprints:SW-Kailh-Hotswap-MX-2.25u -> switches:SW-Kailh-Hotswap-MX-2.25u; symbol MX_Switch:MX-NoLED -> MX-Switch:MX-NoLED
- MX66: value Z -> (none); footprint footprints:SW-Kailh-Hotswap-MX-1.00u -> switches:SW-Kailh-Hotswap-MX-1.00u; symbol MX_Switch:MX-NoLED -> MX-Switch:MX-NoLED
- MX67: value X -> (none); footprint footprints:SW-Kailh-Hotswap-MX-1.00u -> switches:SW-Kailh-Hotswap-MX-1.00u; symbol MX_Switch:MX-NoLED -> MX-Switch:MX-NoLED
- MX68: value C -> (none); footprint footprints:SW-Kailh-Hotswap-MX-1.00u -> switches:SW-Kailh-Hotswap-MX-1.00u; symbol MX_Switch:MX-NoLED -> MX-Switch:MX-NoLED
- MX69: value V -> (none); footprint footprints:SW-Kailh-Hotswap-MX-1.00u -> switches:SW-Kailh-Hotswap-MX-1.00u; symbol MX_Switch:MX-NoLED -> MX-Switch:MX-NoLED
- MX7: value F6 -> (none); footprint footprints:SW-Kailh-Hotswap-MX-1.00u -> switches:SW-Kailh-Hotswap-MX-1.00u; symbol MX_Switch:MX-NoLED -> MX-Switch:MX-NoLED
- MX70: value B -> (none); footprint footprints:SW-Kailh-Hotswap-MX-1.00u -> switches:SW-Kailh-Hotswap-MX-1.00u; symbol MX_Switch:MX-NoLED -> MX-Switch:MX-NoLED
- MX71: value N -> (none); footprint footprints:SW-Kailh-Hotswap-MX-1.00u -> switches:SW-Kailh-Hotswap-MX-1.00u; symbol MX_Switch:MX-NoLED -> MX-Switch:MX-NoLED
- MX72: value M -> (none); footprint footprints:SW-Kailh-Hotswap-MX-1.00u -> switches:SW-Kailh-Hotswap-MX-1.00u; symbol MX_Switch:MX-NoLED -> MX-Switch:MX-NoLED
- MX73: value , -> (none); footprint footprints:SW-Kailh-Hotswap-MX-1.00u -> switches:SW-Kailh-Hotswap-MX-1.00u; symbol MX_Switch:MX-NoLED -> MX-Switch:MX-NoLED
- MX74: value . -> (none); footprint footprints:SW-Kailh-Hotswap-MX-1.00u -> switches:SW-Kailh-Hotswap-MX-1.00u; symbol MX_Switch:MX-NoLED -> MX-Switch:MX-NoLED
- MX75: value / -> (none); footprint footprints:SW-Kailh-Hotswap-MX-1.00u -> switches:SW-Kailh-Hotswap-MX-1.00u; symbol MX_Switch:MX-NoLED -> MX-Switch:MX-NoLED
- MX76: value RShift -> (none); footprint footprints:SW-Kailh-Hotswap-MX-2.75u -> switches:SW-Kailh-Hotswap-MX-2.75u; symbol MX_Switch:MX-NoLED -> MX-Switch:MX-NoLED
- MX77: value Up -> (none); footprint footprints:SW-Kailh-Hotswap-MX-1.00u -> switches:SW-Kailh-Hotswap-MX-1.00u; symbol MX_Switch:MX-NoLED -> MX-Switch:MX-NoLED
- MX78: value LCtrl -> (none); footprint footprints:SW-Kailh-Hotswap-MX-1.25u -> switches:SW-Kailh-Hotswap-MX-1.25u; symbol MX_Switch:MX-NoLED -> MX-Switch:MX-NoLED
- MX79: value Win -> LWin; footprint footprints:SW-Kailh-Hotswap-MX-1.25u -> switches:SW-Kailh-Hotswap-MX-1.25u; symbol MX_Switch:MX-NoLED -> MX-Switch:MX-NoLED
- MX8: value F7 -> (none); footprint footprints:SW-Kailh-Hotswap-MX-1.00u -> switches:SW-Kailh-Hotswap-MX-1.00u; symbol MX_Switch:MX-NoLED -> MX-Switch:MX-NoLED
- MX80: value Alt -> LAlt; footprint footprints:SW-Kailh-Hotswap-MX-1.25u -> switches:SW-Kailh-Hotswap-MX-1.25u; symbol MX_Switch:MX-NoLED -> MX-Switch:MX-NoLED
- MX81: value Space -> (none); footprint footprints:SW-Kailh-Hotswap-MX-6.25u -> switches:SW-Kailh-Hotswap-MX-6.25u; symbol MX_Switch:MX-NoLED -> MX-Switch:MX-NoLED
- MX82: value Alt -> RAlt; footprint footprints:SW-Kailh-Hotswap-MX-1.25u -> switches:SW-Kailh-Hotswap-MX-1.25u; symbol MX_Switch:MX-NoLED -> MX-Switch:MX-NoLED
- MX83: value Win -> RWin; footprint footprints:SW-Kailh-Hotswap-MX-1.25u -> switches:SW-Kailh-Hotswap-MX-1.25u; symbol MX_Switch:MX-NoLED -> MX-Switch:MX-NoLED
- MX84: value Fn -> (none); footprint footprints:SW-Kailh-Hotswap-MX-1.25u -> switches:SW-Kailh-Hotswap-MX-1.25u; symbol MX_Switch:MX-NoLED -> MX-Switch:MX-NoLED
- MX85: value RCtrl -> (none); footprint footprints:SW-Kailh-Hotswap-MX-1.25u -> switches:SW-Kailh-Hotswap-MX-1.25u; symbol MX_Switch:MX-NoLED -> MX-Switch:MX-NoLED
- MX86: value Left -> (none); footprint footprints:SW-Kailh-Hotswap-MX-1.00u -> switches:SW-Kailh-Hotswap-MX-1.00u; symbol MX_Switch:MX-NoLED -> MX-Switch:MX-NoLED
- MX87: value Down -> (none); footprint footprints:SW-Kailh-Hotswap-MX-1.00u -> switches:SW-Kailh-Hotswap-MX-1.00u; symbol MX_Switch:MX-NoLED -> MX-Switch:MX-NoLED
- MX88: value Right -> (none); footprint footprints:SW-Kailh-Hotswap-MX-1.00u -> switches:SW-Kailh-Hotswap-MX-1.00u; symbol MX_Switch:MX-NoLED -> MX-Switch:MX-NoLED
- MX9: value F8 -> (none); footprint footprints:SW-Kailh-Hotswap-MX-1.00u -> switches:SW-Kailh-Hotswap-MX-1.00u; symbol MX_Switch:MX-NoLED -> MX-Switch:MX-NoLED

Commit message: Routed matrix and MCU
Parts:
- D10, D11, D12, D13, D14, D15, D16, D17, D18, D19, D2, D20, D21, D22, D23, D24, D25, D26, D27, D28, D29, D3, D30, D31, D32, D33, D34, D35, D36, D37, D38, D39, D4, D40, D41, D42, D43, D44, D45, D46, D47, D48, D49, D5, D50, D51, D52, D53, D54, D55, D56, D57, D58, D59, D6, D60, D61, D62, D63, D64, D65, D66, D67, D68, D69, D7, D70, D71, D72, D73, D74, D75, D76, D77, D78, D79, D8, D80, D81, D82, D83, D84, D85, D86, D87, D88, D9: value (none) -> D_Small
- MX1, MX79, MX80, MX82, MX83: now left out of the parts list
- MX10: value (none) -> F9; now left out of the parts list
- MX11: value (none) -> F10; now left out of the parts list
- MX12: value (none) -> F11; now left out of the parts list
- MX13: value (none) -> F12; now left out of the parts list
- MX14: value (none) -> F13; now left out of the parts list
- MX15: value (none) -> PrtSc; now left out of the parts list
- MX16: value (none) -> ScrLck; now left out of the parts list
- MX17: value (none) -> Pause; now left out of the parts list
- MX18: value (none) -> ~; now left out of the parts list
- MX19: value (none) -> 1; now left out of the parts list
- MX2: value (none) -> F1; now left out of the parts list
- MX20: value (none) -> 2; now left out of the parts list
- MX21: value (none) -> 3; now left out of the parts list
- MX22: value (none) -> 4; now left out of the parts list
- MX23: value (none) -> 5; now left out of the parts list
- MX24: value (none) -> 6; now left out of the parts list
- MX25: value (none) -> 7; now left out of the parts list
- MX26: value (none) -> 8; now left out of the parts list
- MX27: value (none) -> 9; now left out of the parts list
- MX28: value (none) -> 0; now left out of the parts list
- MX29: value (none) -> -; now left out of the parts list
- MX3: value (none) -> F2; now left out of the parts list
- MX30: value (none) -> +; now left out of the parts list
- MX31: value (none) -> Bck; now left out of the parts list
- MX32: value (none) -> Insert; now left out of the parts list
- MX33: value (none) -> Home; now left out of the parts list
- MX34: value (none) -> PgUp; now left out of the parts list
- MX35: value (none) -> Tab; now left out of the parts list
- MX36: value (none) -> Q; now left out of the parts list
- MX37: value (none) -> W; now left out of the parts list
- MX38: value (none) -> E; now left out of the parts list
- MX39: value (none) -> R; now left out of the parts list
- MX4: value (none) -> F3; now left out of the parts list
- MX40: value (none) -> T; now left out of the parts list
- MX41: value (none) -> Y; now left out of the parts list
- MX42: value (none) -> U; now left out of the parts list
- MX43: value (none) -> I; now left out of the parts list
- MX44: value (none) -> O; now left out of the parts list
- MX45: value (none) -> P; now left out of the parts list
- MX46: value (none) -> [; now left out of the parts list
- MX47: value (none) -> ]; now left out of the parts list
- MX48: value (none) -> \; footprint switches:SW-Kailh-Hotswap-MX-1.00u -> switches:SW-Kailh-Hotswap-MX-1.50u; now left out of the parts list
- MX49: value (none) -> Delete; now left out of the parts list
- MX5: value (none) -> F4; now left out of the parts list
- MX50: value (none) -> End; now left out of the parts list
- MX51: value (none) -> PgDn; now left out of the parts list
- MX52: value (none) -> Caps; now left out of the parts list
- MX53: value (none) -> A; now left out of the parts list
- MX54: value (none) -> S; now left out of the parts list
- MX55: value (none) -> D; now left out of the parts list
- MX56: value (none) -> F; now left out of the parts list
- MX57: value (none) -> G; now left out of the parts list
- MX58: value (none) -> H; now left out of the parts list
- MX59: value (none) -> J; now left out of the parts list
- MX6: value (none) -> F5; now left out of the parts list
- MX60: value (none) -> K; now left out of the parts list
- MX61: value (none) -> L; now left out of the parts list
- MX62: value (none) -> ;; now left out of the parts list
- MX63: value (none) -> '; now left out of the parts list
- MX64: value (none) -> Enter; now left out of the parts list
- MX65: value (none) -> LShift; now left out of the parts list
- MX66: value (none) -> Z; now left out of the parts list
- MX67: value (none) -> X; now left out of the parts list
- MX68: value (none) -> C; now left out of the parts list
- MX69: value (none) -> V; now left out of the parts list
- MX7: value (none) -> F6; now left out of the parts list
- MX70: value (none) -> B; now left out of the parts list
- MX71: value (none) -> N; now left out of the parts list
- MX72: value (none) -> M; now left out of the parts list
- MX73: value (none) -> ,; now left out of the parts list
- MX74: value (none) -> .; now left out of the parts list
- MX75: value (none) -> /; now left out of the parts list
- MX76: value (none) -> RShift; now left out of the parts list
- MX77: value (none) -> Up; now left out of the parts list
- MX78: value (none) -> LCtrl; now left out of the parts list
- MX8: value (none) -> F7; now left out of the parts list
- MX81: value (none) -> Space; now left out of the parts list
- MX84: value (none) -> Fn; now left out of the parts list
- MX85: value (none) -> RCtrl; now left out of the parts list
- MX86: value (none) -> Left; now left out of the parts list
- MX87: value (none) -> Down; now left out of the parts list
- MX88: value (none) -> Right; now left out of the parts list
- MX9: value (none) -> F8; now left out of the parts list

Commit message: update
Parts:
- removed MX1: Esc, switches:SW-Kailh-Hotswap-MX-1.00u, symbol MX-Switch:MX-NoLED
- removed MX10: F9, switches:SW-Kailh-Hotswap-MX-1.00u, symbol MX-Switch:MX-NoLED
- removed MX11: F10, switches:SW-Kailh-Hotswap-MX-1.00u, symbol MX-Switch:MX-NoLED
- removed MX12: F11, switches:SW-Kailh-Hotswap-MX-1.00u, symbol MX-Switch:MX-NoLED
- removed MX13: F12, switches:SW-Kailh-Hotswap-MX-1.00u, symbol MX-Switch:MX-NoLED
- removed MX14: F13, switches:SW-Kailh-Hotswap-MX-1.00u, symbol MX-Switch:MX-NoLED
- removed MX15: PrtSc, switches:SW-Kailh-Hotswap-MX-1.00u, symbol MX-Switch:MX-NoLED
- removed MX16: ScrLck, switches:SW-Kailh-Hotswap-MX-1.00u, symbol MX-Switch:MX-NoLED
- removed MX17: Pause, switches:SW-Kailh-Hotswap-MX-1.00u, symbol MX-Switch:MX-NoLED
- removed MX18: ~, switches:SW-Kailh-Hotswap-MX-1.00u, symbol MX-Switch:MX-NoLED
- removed MX19: 1, switches:SW-Kailh-Hotswap-MX-1.00u, symbol MX-Switch:MX-NoLED
- removed MX2: F1, switches:SW-Kailh-Hotswap-MX-1.00u, symbol MX-Switch:MX-NoLED
- removed MX20: 2, switches:SW-Kailh-Hotswap-MX-1.00u, symbol MX-Switch:MX-NoLED
- removed MX21: 3, switches:SW-Kailh-Hotswap-MX-1.00u, symbol MX-Switch:MX-NoLED
- removed MX22: 4, switches:SW-Kailh-Hotswap-MX-1.00u, symbol MX-Switch:MX-NoLED
- removed MX23: 5, switches:SW-Kailh-Hotswap-MX-1.00u, symbol MX-Switch:MX-NoLED
- removed MX24: 6, switches:SW-Kailh-Hotswap-MX-1.00u, symbol MX-Switch:MX-NoLED
- removed MX25: 7, switches:SW-Kailh-Hotswap-MX-1.00u, symbol MX-Switch:MX-NoLED
- removed MX26: 8, switches:SW-Kailh-Hotswap-MX-1.00u, symbol MX-Switch:MX-NoLED
- removed MX27: 9, switches:SW-Kailh-Hotswap-MX-1.00u, symbol MX-Switch:MX-NoLED
- removed MX28: 0, switches:SW-Kailh-Hotswap-MX-1.00u, symbol MX-Switch:MX-NoLED
- removed MX29: -, switches:SW-Kailh-Hotswap-MX-1.00u, symbol MX-Switch:MX-NoLED
- removed MX3: F2, switches:SW-Kailh-Hotswap-MX-1.00u, symbol MX-Switch:MX-NoLED
- removed MX30: +, switches:SW-Kailh-Hotswap-MX-1.00u, symbol MX-Switch:MX-NoLED
- removed MX31: Bck, switches:SW-Kailh-Hotswap-MX-2.00u, symbol MX-Switch:MX-NoLED
- removed MX32: Insert, switches:SW-Kailh-Hotswap-MX-1.00u, symbol MX-Switch:MX-NoLED
- removed MX33: Home, switches:SW-Kailh-Hotswap-MX-1.00u, symbol MX-Switch:MX-NoLED
- removed MX34: PgUp, switches:SW-Kailh-Hotswap-MX-1.00u, symbol MX-Switch:MX-NoLED
- removed MX35: Tab, switches:SW-Kailh-Hotswap-MX-1.50u, symbol MX-Switch:MX-NoLED
- removed MX36: Q, switches:SW-Kailh-Hotswap-MX-1.00u, symbol MX-Switch:MX-NoLED
- removed MX37: W, switches:SW-Kailh-Hotswap-MX-1.00u, symbol MX-Switch:MX-NoLED
- removed MX38: E, switches:SW-Kailh-Hotswap-MX-1.00u, symbol MX-Switch:MX-NoLED
- removed MX39: R, switches:SW-Kailh-Hotswap-MX-1.00u, symbol MX-Switch:MX-NoLED
- removed MX4: F3, switches:SW-Kailh-Hotswap-MX-1.00u, symbol MX-Switch:MX-NoLED
- removed MX40: T, switches:SW-Kailh-Hotswap-MX-1.00u, symbol MX-Switch:MX-NoLED
- removed MX41: Y, switches:SW-Kailh-Hotswap-MX-1.00u, symbol MX-Switch:MX-NoLED
- removed MX42: U, switches:SW-Kailh-Hotswap-MX-1.00u, symbol MX-Switch:MX-NoLED
- removed MX43: I, switches:SW-Kailh-Hotswap-MX-1.00u, symbol MX-Switch:MX-NoLED
- removed MX44: O, switches:SW-Kailh-Hotswap-MX-1.00u, symbol MX-Switch:MX-NoLED
- removed MX45: P, switches:SW-Kailh-Hotswap-MX-1.00u, symbol MX-Switch:MX-NoLED
- removed MX46: [, switches:SW-Kailh-Hotswap-MX-1.00u, symbol MX-Switch:MX-NoLED
- removed MX47: ], switches:SW-Kailh-Hotswap-MX-1.00u, symbol MX-Switch:MX-NoLED
- removed MX48: \, switches:SW-Kailh-Hotswap-MX-1.50u, symbol MX-Switch:MX-NoLED
- removed MX49: Delete, switches:SW-Kailh-Hotswap-MX-1.00u, symbol MX-Switch:MX-NoLED
- removed MX5: F4, switches:SW-Kailh-Hotswap-MX-1.00u, symbol MX-Switch:MX-NoLED
- removed MX50: End, switches:SW-Kailh-Hotswap-MX-1.00u, symbol MX-Switch:MX-NoLED
- removed MX51: PgDn, switches:SW-Kailh-Hotswap-MX-1.00u, symbol MX-Switch:MX-NoLED
- removed MX52: Caps, switches:SW-Kailh-Hotswap-MX-1.75u, symbol MX-Switch:MX-NoLED
- removed MX53: A, switches:SW-Kailh-Hotswap-MX-1.00u, symbol MX-Switch:MX-NoLED
- removed MX54: S, switches:SW-Kailh-Hotswap-MX-1.00u, symbol MX-Switch:MX-NoLED
- removed MX55: D, switches:SW-Kailh-Hotswap-MX-1.00u, symbol MX-Switch:MX-NoLED
- removed MX56: F, switches:SW-Kailh-Hotswap-MX-1.00u, symbol MX-Switch:MX-NoLED
- removed MX57: G, switches:SW-Kailh-Hotswap-MX-1.00u, symbol MX-Switch:MX-NoLED
- removed MX58: H, switches:SW-Kailh-Hotswap-MX-1.00u, symbol MX-Switch:MX-NoLED
- removed MX59: J, switches:SW-Kailh-Hotswap-MX-1.00u, symbol MX-Switch:MX-NoLED
- removed MX6: F5, switches:SW-Kailh-Hotswap-MX-1.00u, symbol MX-Switch:MX-NoLED
- removed MX60: K, switches:SW-Kailh-Hotswap-MX-1.00u, symbol MX-Switch:MX-NoLED
- removed MX61: L, switches:SW-Kailh-Hotswap-MX-1.00u, symbol MX-Switch:MX-NoLED
- removed MX62: ;, switches:SW-Kailh-Hotswap-MX-1.00u, symbol MX-Switch:MX-NoLED
- removed MX63: ', switches:SW-Kailh-Hotswap-MX-1.00u, symbol MX-Switch:MX-NoLED
- removed MX64: Enter, switches:SW-Kailh-Hotswap-MX-2.25u, symbol MX-Switch:MX-NoLED
- removed MX65: LShift, switches:SW-Kailh-Hotswap-MX-2.25u, symbol MX-Switch:MX-NoLED
- removed MX66: Z, switches:SW-Kailh-Hotswap-MX-1.00u, symbol MX-Switch:MX-NoLED
- removed MX67: X, switches:SW-Kailh-Hotswap-MX-1.00u, symbol MX-Switch:MX-NoLED
- removed MX68: C, switches:SW-Kailh-Hotswap-MX-1.00u, symbol MX-Switch:MX-NoLED
- removed MX69: V, switches:SW-Kailh-Hotswap-MX-1.00u, symbol MX-Switch:MX-NoLED
- removed MX7: F6, switches:SW-Kailh-Hotswap-MX-1.00u, symbol MX-Switch:MX-NoLED
- removed MX70: B, switches:SW-Kailh-Hotswap-MX-1.00u, symbol MX-Switch:MX-NoLED
- removed MX71: N, switches:SW-Kailh-Hotswap-MX-1.00u, symbol MX-Switch:MX-NoLED
- removed MX72: M, switches:SW-Kailh-Hotswap-MX-1.00u, symbol MX-Switch:MX-NoLED
- removed MX73: ,, switches:SW-Kailh-Hotswap-MX-1.00u, symbol MX-Switch:MX-NoLED
- removed MX74: ., switches:SW-Kailh-Hotswap-MX-1.00u, symbol MX-Switch:MX-NoLED
- removed MX75: /, switches:SW-Kailh-Hotswap-MX-1.00u, symbol MX-Switch:MX-NoLED
- removed MX76: RShift, switches:SW-Kailh-Hotswap-MX-2.75u, symbol MX-Switch:MX-NoLED
- removed MX77: Up, switches:SW-Kailh-Hotswap-MX-1.00u, symbol MX-Switch:MX-NoLED
- removed MX78: LCtrl, switches:SW-Kailh-Hotswap-MX-1.25u, symbol MX-Switch:MX-NoLED
- removed MX79: LWin, switches:SW-Kailh-Hotswap-MX-1.25u, symbol MX-Switch:MX-NoLED
- removed MX8: F7, switches:SW-Kailh-Hotswap-MX-1.00u, symbol MX-Switch:MX-NoLED
- removed MX80: LAlt, switches:SW-Kailh-Hotswap-MX-1.25u, symbol MX-Switch:MX-NoLED
- removed MX81: Space, switches:SW-Kailh-Hotswap-MX-6.25u, symbol MX-Switch:MX-NoLED
- removed MX82: RAlt, switches:SW-Kailh-Hotswap-MX-1.25u, symbol MX-Switch:MX-NoLED
- removed MX83: RWin, switches:SW-Kailh-Hotswap-MX-1.25u, symbol MX-Switch:MX-NoLED
- removed MX84: Fn, switches:SW-Kailh-Hotswap-MX-1.25u, symbol MX-Switch:MX-NoLED
- removed MX85: RCtrl, switches:SW-Kailh-Hotswap-MX-1.25u, symbol MX-Switch:MX-NoLED
- removed MX86: Left, switches:SW-Kailh-Hotswap-MX-1.00u, symbol MX-Switch:MX-NoLED
- removed MX87: Down, switches:SW-Kailh-Hotswap-MX-1.00u, symbol MX-Switch:MX-NoLED
- removed MX88: Right, switches:SW-Kailh-Hotswap-MX-1.00u, symbol MX-Switch:MX-NoLED
- removed MX9: F8, switches:SW-Kailh-Hotswap-MX-1.00u, symbol MX-Switch:MX-NoLED
- added D89: 1N4148W, Diode_SMD:D_SOD-123, symbol Device:D_Small
- added MX1: Esc, SW-MX:SW-Kailh-Hotswap-MX-1.00u, symbol MX_Switch:MX-NoLED
- added MX10: F9, SW-MX:SW-Kailh-Hotswap-MX-1.00u, symbol MX_Switch:MX-NoLED
- added MX11: F10, SW-MX:SW-Kailh-Hotswap-MX-1.00u, symbol MX_Switch:MX-NoLED
- added MX12: F11, SW-MX:SW-Kailh-Hotswap-MX-1.00u, symbol MX_Switch:MX-NoLED
- added MX13: F12, SW-MX:SW-Kailh-Hotswap-MX-1.00u, symbol MX_Switch:MX-NoLED
- added MX14: F13, SW-MX:SW-Kailh-Hotswap-MX-1.00u, symbol MX_Switch:MX-NoLED
- added MX15: PrtSc, SW-MX:SW-Kailh-Hotswap-MX-1.00u, symbol MX_Switch:MX-NoLED
- added MX16: S Lck, SW-MX:SW-Kailh-Hotswap-MX-1.00u, symbol MX_Switch:MX-NoLED
- added MX17: Pause, SW-MX:SW-Kailh-Hotswap-MX-1.00u, symbol MX_Switch:MX-NoLED
- added MX18: ~, SW-MX:SW-Kailh-Hotswap-MX-1.00u, symbol MX_Switch:MX-NoLED
- added MX19: 1, SW-MX:SW-Kailh-Hotswap-MX-1.00u, symbol MX_Switch:MX-NoLED
- added MX2: F1, SW-MX:SW-Kailh-Hotswap-MX-1.00u, symbol MX_Switch:MX-NoLED
- added MX20: 2, SW-MX:SW-Kailh-Hotswap-MX-1.00u, symbol MX_Switch:MX-NoLED
- added MX21: 3, SW-MX:SW-Kailh-Hotswap-MX-1.00u, symbol MX_Switch:MX-NoLED
- added MX22: 4, SW-MX:SW-Kailh-Hotswap-MX-1.00u, symbol MX_Switch:MX-NoLED
- added MX23: 5, SW-MX:SW-Kailh-Hotswap-MX-1.00u, symbol MX_Switch:MX-NoLED
- added MX24: 6, SW-MX:SW-Kailh-Hotswap-MX-1.00u, symbol MX_Switch:MX-NoLED
- added MX25: 7, SW-MX:SW-Kailh-Hotswap-MX-1.00u, symbol MX_Switch:MX-NoLED
- added MX26: 8, SW-MX:SW-Kailh-Hotswap-MX-1.00u, symbol MX_Switch:MX-NoLED
- added MX27: 9, SW-MX:SW-Kailh-Hotswap-MX-1.00u, symbol MX_Switch:MX-NoLED
- added MX28: 0, SW-MX:SW-Kailh-Hotswap-MX-1.00u, symbol MX_Switch:MX-NoLED
- added MX29: -, SW-MX:SW-Kailh-Hotswap-MX-1.00u, symbol MX_Switch:MX-NoLED
- added MX3: F2, SW-MX:SW-Kailh-Hotswap-MX-1.00u, symbol MX_Switch:MX-NoLED
- added MX30: =, SW-MX:SW-Kailh-Hotswap-MX-1.00u, symbol MX_Switch:MX-NoLED
- added MX31: Backspace, SW-MX:SW-Kailh-Hotswap-MX-2.00u, symbol MX_Switch:MX-NoLED
- added MX32: Insert, SW-MX:SW-Kailh-Hotswap-MX-1.00u, symbol MX_Switch:MX-NoLED
- added MX33: Home, SW-MX:SW-Kailh-Hotswap-MX-1.00u, symbol MX_Switch:MX-NoLED
- added MX34: PgUp, SW-MX:SW-Kailh-Hotswap-MX-1.00u, symbol MX_Switch:MX-NoLED
- added MX35: Tab, SW-MX:SW-Kailh-Hotswap-MX-1.50u, symbol MX_Switch:MX-NoLED
- added MX36: Q, SW-MX:SW-Kailh-Hotswap-MX-1.00u, symbol MX_Switch:MX-NoLED
- added MX37: W, SW-MX:SW-Kailh-Hotswap-MX-1.00u, symbol MX_Switch:MX-NoLED
- added MX38: E, SW-MX:SW-Kailh-Hotswap-MX-1.00u, symbol MX_Switch:MX-NoLED
- added MX39: R, SW-MX:SW-Kailh-Hotswap-MX-1.00u, symbol MX_Switch:MX-NoLED
- added MX4: F3, SW-MX:SW-Kailh-Hotswap-MX-1.00u, symbol MX_Switch:MX-NoLED
- added MX40: T, SW-MX:SW-Kailh-Hotswap-MX-1.00u, symbol MX_Switch:MX-NoLED
- added MX41: Y, SW-MX:SW-Kailh-Hotswap-MX-1.00u, symbol MX_Switch:MX-NoLED
- added MX42: U, SW-MX:SW-Kailh-Hotswap-MX-1.00u, symbol MX_Switch:MX-NoLED
- added MX43: I, SW-MX:SW-Kailh-Hotswap-MX-1.00u, symbol MX_Switch:MX-NoLED
- added MX44: O, SW-MX:SW-Kailh-Hotswap-MX-1.00u, symbol MX_Switch:MX-NoLED
- added MX45: P, SW-MX:SW-Kailh-Hotswap-MX-1.00u, symbol MX_Switch:MX-NoLED
- added MX46: [, SW-MX:SW-Kailh-Hotswap-MX-1.00u, symbol MX_Switch:MX-NoLED
- added MX47: ], SW-MX:SW-Kailh-Hotswap-MX-1.00u, symbol MX_Switch:MX-NoLED
- added MX48: \, SW-MX:SW-Kailh-Hotswap-MX-1.50u, symbol MX_Switch:MX-NoLED
- added MX49: Delete, SW-MX:SW-Kailh-Hotswap-MX-1.00u, symbol MX_Switch:MX-NoLED
- added MX5: F4, SW-MX:SW-Kailh-Hotswap-MX-1.00u, symbol MX_Switch:MX-NoLED
- added MX50: End, SW-MX:SW-Kailh-Hotswap-MX-1.00u, symbol MX_Switch:MX-NoLED
- added MX51: PgDn, SW-MX:SW-Kailh-Hotswap-MX-1.00u, symbol MX_Switch:MX-NoLED
- added MX52: Caps, SW-MX:SW-Kailh-Hotswap-MX-1.75u, symbol MX_Switch:MX-NoLED
- added MX53: A, SW-MX:SW-Kailh-Hotswap-MX-1.00u, symbol MX_Switch:MX-NoLED
- added MX54: S, SW-MX:SW-Kailh-Hotswap-MX-1.00u, symbol MX_Switch:MX-NoLED
- added MX55: D, SW-MX:SW-Kailh-Hotswap-MX-1.00u, symbol MX_Switch:MX-NoLED
- added MX56: F, SW-MX:SW-Kailh-Hotswap-MX-1.00u, symbol MX_Switch:MX-NoLED
- added MX57: G, SW-MX:SW-Kailh-Hotswap-MX-1.00u, symbol MX_Switch:MX-NoLED
- added MX58: H, SW-MX:SW-Kailh-Hotswap-MX-1.00u, symbol MX_Switch:MX-NoLED
- added MX59: J, SW-MX:SW-Kailh-Hotswap-MX-1.00u, symbol MX_Switch:MX-NoLED
- added MX6: F5, SW-MX:SW-Kailh-Hotswap-MX-1.00u, symbol MX_Switch:MX-NoLED
- added MX60: K, SW-MX:SW-Kailh-Hotswap-MX-1.00u, symbol MX_Switch:MX-NoLED
- added MX61: L, SW-MX:SW-Kailh-Hotswap-MX-1.00u, symbol MX_Switch:MX-NoLED
- added MX62: ;, SW-MX:SW-Kailh-Hotswap-MX-1.00u, symbol MX_Switch:MX-NoLED
- added MX63: ', SW-MX:SW-Kailh-Hotswap-MX-1.00u, symbol MX_Switch:MX-NoLED
- added MX64: Enter, SW-MX:SW-Kailh-Hotswap-MX-2.25u, symbol MX_Switch:MX-NoLED
- added MX65: L-Shift, SW-MX:SW-Kailh-Hotswap-MX-2.25u, symbol MX_Switch:MX-NoLED
- added MX66: Z, SW-MX:SW-Kailh-Hotswap-MX-1.00u, symbol MX_Switch:MX-NoLED
- added MX67: X, SW-MX:SW-Kailh-Hotswap-MX-1.00u, symbol MX_Switch:MX-NoLED
- added MX68: C, SW-MX:SW-Kailh-Hotswap-MX-1.00u, symbol MX_Switch:MX-NoLED
- added MX69: V, SW-MX:SW-Kailh-Hotswap-MX-1.00u, symbol MX_Switch:MX-NoLED
- added MX7: F6, SW-MX:SW-Kailh-Hotswap-MX-1.00u, symbol MX_Switch:MX-NoLED
- added MX70: B, SW-MX:SW-Kailh-Hotswap-MX-1.00u, symbol MX_Switch:MX-NoLED
- added MX71: N, SW-MX:SW-Kailh-Hotswap-MX-1.00u, symbol MX_Switch:MX-NoLED
- added MX72: M, SW-MX:SW-Kailh-Hotswap-MX-1.00u, symbol MX_Switch:MX-NoLED
- added MX73: {lt}, SW-MX:SW-Kailh-Hotswap-MX-1.00u, symbol MX_Switch:MX-NoLED
- added MX74: >, SW-MX:SW-Kailh-Hotswap-MX-1.00u, symbol MX_Switch:MX-NoLED
- added MX75: /, SW-MX:SW-Kailh-Hotswap-MX-1.00u, symbol MX_Switch:MX-NoLED
- added MX76: R-Shift, SW-MX:SW-Kailh-Hotswap-MX-1.75u, symbol MX_Switch:MX-NoLED
- added MX77: Fn, SW-MX:SW-Kailh-Hotswap-MX-1.00u, symbol MX_Switch:MX-NoLED
- added MX78: Up, SW-MX:SW-Kailh-Hotswap-MX-1.00u, symbol MX_Switch:MX-NoLED
- added MX79: L-Ctrl, SW-MX:SW-Kailh-Hotswap-MX-1.25u, symbol MX_Switch:MX-NoLED
- added MX8: F7, SW-MX:SW-Kailh-Hotswap-MX-1.00u, symbol MX_Switch:MX-NoLED
- added MX80: L-Mod, SW-MX:SW-Kailh-Hotswap-MX-1.25u, symbol MX_Switch:MX-NoLED
- added MX81: L-Alt, SW-MX:SW-Kailh-Hotswap-MX-1.25u, symbol MX_Switch:MX-NoLED
- added MX82: Space, SW-MX:SW-Kailh-Hotswap-MX-6.25u, symbol MX_Switch:MX-NoLED
- added MX83: R-Alt, SW-MX:SW-Kailh-Hotswap-MX-1.25u, symbol MX_Switch:MX-NoLED
- added MX84: R-Mod, SW-MX:SW-Kailh-Hotswap-MX-1.25u, symbol MX_Switch:MX-NoLED
- added MX85: Fn, SW-MX:SW-Kailh-Hotswap-MX-1.25u, symbol MX_Switch:MX-NoLED
- added MX86: R-Ctrl, SW-MX:SW-Kailh-Hotswap-MX-1.25u, symbol MX_Switch:MX-NoLED
- added MX87: Left, SW-MX:SW-Kailh-Hotswap-MX-1.00u, symbol MX_Switch:MX-NoLED
- added MX88: Down, SW-MX:SW-Kailh-Hotswap-MX-1.00u, symbol MX_Switch:MX-NoLED
- added MX89: Right, SW-MX:SW-Kailh-Hotswap-MX-1.00u, symbol MX_Switch:MX-NoLED
- added MX9: F8, SW-MX:SW-Kailh-Hotswap-MX-1.00u, symbol MX_Switch:MX-NoLED
- D1, D10, D11, D12, D13, D14, D15, D16, D17, D18, D19, D2, D20, D21, D22, D23, D24, D25, D26, D27, D28, D29, D3, D30, D31, D32, D33, D34, D35, D36, D37, D38, D39, D4, D40, D41, D42, D43, D44, D45, D46, D47, D48, D49, D5, D50, D51, D52, D53, D54, D55, D56, D57, D58, D59, D6, D60, D61, D62, D63, D64, D65, D66, D67, D68, D69, D7, D70, D71, D72, D73, D74, D75, D76, D77, D78, D79, D8, D80, D81, D82, D83, D84, D85, D86, D87, D88, D9: value D_Small -> 1N4148W; footprint diodes:D-0603-1608 -> Diode_SMD:D_SOD-123
Connections:
- net COL0: now also MX1.1 (COL), MX18.1 (COL), MX35.1 (COL), MX52.1 (COL), MX65.1 (COL), MX79.1 (COL)
- net COL1: now also MX19.1 (COL), MX2.1 (COL), MX36.1 (COL), MX53.1 (COL), MX80.1 (COL)
- net COL10: now also MX11.1 (COL), MX28.1 (COL), MX45.1 (COL), MX62.1 (COL), MX74.1 (COL), MX83.1 (COL)
- net COL11: now also MX12.1 (COL), MX29.1 (COL), MX46.1 (COL), MX63.1 (COL), MX75.1 (COL), MX84.1 (COL)
- net COL12: now also MX13.1 (COL), MX30.1 (COL), MX47.1 (COL), MX76.1 (COL), MX85.1 (COL)
- net COL13: now also MX14.1 (COL), MX31.1 (COL), MX48.1 (COL), MX64.1 (COL), MX77.1 (COL), MX86.1 (COL)
- net COL14: now also MX15.1 (COL), MX32.1 (COL), MX49.1 (COL), MX87.1 (COL)
- net COL15: now also MX16.1 (COL), MX33.1 (COL), MX50.1 (COL), MX78.1 (COL), MX88.1 (COL)
- net COL16: now also MX17.1 (COL), MX34.1 (COL), MX51.1 (COL), MX89.1 (COL)
- net COL2: now also MX20.1 (COL), MX3.1 (COL), MX37.1 (COL), MX54.1 (COL), MX66.1 (COL), MX81.1 (COL)
- net COL3: now also MX21.1 (COL), MX38.1 (COL), MX4.1 (COL), MX55.1 (COL), MX67.1 (COL)
- net COL4: now also MX22.1 (COL), MX39.1 (COL), MX5.1 (COL), MX56.1 (COL), MX68.1 (COL)
- net COL5: now also MX23.1 (COL), MX40.1 (COL), MX57.1 (COL), MX6.1 (COL), MX69.1 (COL)
- net COL6: now also MX24.1 (COL), MX41.1 (COL), MX58.1 (COL), MX7.1 (COL), MX70.1 (COL), MX82.1 (COL)
- net COL7: now also MX25.1 (COL), MX42.1 (COL), MX59.1 (COL), MX71.1 (COL), MX8.1 (COL)
- net COL8: now also MX26.1 (COL), MX43.1 (COL), MX60.1 (COL), MX72.1 (COL), MX9.1 (COL)
- net COL9: now also MX10.1 (COL), MX27.1 (COL), MX44.1 (COL), MX61.1 (COL), MX73.1 (COL)
- net ROW4: now also D78.1 (K)
- net ROW5: now also D89.1 (K); no longer D78.1 (K)
- net at D21.2 (A): now also MX21.2 (ROW)
- net at D64.2 (A): now also MX64.2 (ROW)
- net at D58.2 (A): now also MX58.2 (ROW)
- net at D29.2 (A): now also MX29.2 (ROW)
- net at D51.2 (A): now also MX51.2 (ROW)
- net at D71.2 (A): now also MX71.2 (ROW)
- net at D88.2 (A): now also MX88.2 (ROW)
- net at D34.2 (A): now also MX34.2 (ROW)
- net at D49.2 (A): now also MX49.2 (ROW)
- net at D85.2 (A): now also MX85.2 (ROW)
- net at D74.2 (A): now also MX74.2 (ROW)
- net at D81.2 (A): now also MX81.2 (ROW)
- net at D18.2 (A): now also MX18.2 (ROW)
- net at D47.2 (A): now also MX47.2 (ROW)
- net at D13.2 (A): now also MX13.2 (ROW)
- net at D43.2 (A): now also MX43.2 (ROW)
- net at D67.2 (A): now also MX67.2 (ROW)
- net at D32.2 (A): now also MX32.2 (ROW)
- net at D38.2 (A): now also MX38.2 (ROW)
- net at D12.2 (A): now also MX12.2 (ROW)
- net at D56.2 (A): now also MX56.2 (ROW)
- net at D69.2 (A): now also MX69.2 (ROW)
- net at D14.2 (A): now also MX14.2 (ROW)
- net at D54.2 (A): now also MX54.2 (ROW)
- net at D84.2 (A): now also MX84.2 (ROW)
- net at D5.2 (A): now also MX5.2 (ROW)
- net at D6.2 (A): now also MX6.2 (ROW)
- net at D11.2 (A): now also MX11.2 (ROW)
- net at D28.2 (A): now also MX28.2 (ROW)
- net at D78.2 (A): now also MX78.2 (ROW)
- net at D9.2 (A): now also MX9.2 (ROW)
- net at D8.2 (A): now also MX8.2 (ROW)
- net at D83.2 (A): now also MX83.2 (ROW)
- net at D60.2 (A): now also MX60.2 (ROW)
- net at D24.2 (A): now also MX24.2 (ROW)
- net at D40.2 (A): now also MX40.2 (ROW)
- net at D62.2 (A): now also MX62.2 (ROW)
- net at D19.2 (A): now also MX19.2 (ROW)
- net at D41.2 (A): now also MX41.2 (ROW)
- net at D55.2 (A): now also MX55.2 (ROW)
- net at D45.2 (A): now also MX45.2 (ROW)
- net at D72.2 (A): now also MX72.2 (ROW)
- net at D86.2 (A): now also MX86.2 (ROW)
- net at D16.2 (A): now also MX16.2 (ROW)
- net at D76.2 (A): now also MX76.2 (ROW)
- net at D48.2 (A): now also MX48.2 (ROW)
- net at D35.2 (A): now also MX35.2 (ROW)
- net at D15.2 (A): now also MX15.2 (ROW)
- net at D25.2 (A): now also MX25.2 (ROW)
- net at D65.2 (A): now also MX65.2 (ROW)
- net at D79.2 (A): now also MX79.2 (ROW)
- net at D70.2 (A): now also MX70.2 (ROW)
- net at D75.2 (A): now also MX75.2 (ROW)
- net at D37.2 (A): now also MX37.2 (ROW)
- net at D53.2 (A): now also MX53.2 (ROW)
- net at D23.2 (A): now also MX23.2 (ROW)
- net at D42.2 (A): now also MX42.2 (ROW)
- net at D36.2 (A): now also MX36.2 (ROW)
- net at D82.2 (A): now also MX82.2 (ROW)
- net at D77.2 (A): now also MX77.2 (ROW)
- net at D80.2 (A): now also MX80.2 (ROW)
- net at D87.2 (A): now also MX87.2 (ROW)
- net at D52.2 (A): now also MX52.2 (ROW)
- net at D39.2 (A): now also MX39.2 (ROW)
- net at D73.2 (A): now also MX73.2 (ROW)
- net at D30.2 (A): now also MX30.2 (ROW)
- net at D50.2 (A): now also MX50.2 (ROW)
- net at D3.2 (A): now also MX3.2 (ROW)
- net at D26.2 (A): now also MX26.2 (ROW)
- net at D27.2 (A): now also MX27.2 (ROW)
- net at D57.2 (A): now also MX57.2 (ROW)
- net at D33.2 (A): now also MX33.2 (ROW)
- new net: D89.2 (A), MX89.2 (ROW)
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Other:
- note added: "*split right shift *extra F13 key"
- company: (none) -> rothman
- title: (none) -> Switch Matrix

Commit message: PCB layout complete
Parts:
- MX1, MX10, MX11, MX12, MX13, MX14, MX15, MX16, MX17, MX18, MX19, MX2, MX20, MX21, MX22, MX23, MX24, MX25, MX26, MX27, MX28, MX29, MX3, MX30, MX32, MX33, MX34, MX36, MX37, MX38, MX39, MX4, MX40, MX41, MX42, MX43, MX44, MX45, MX46, MX47, MX49, MX5, MX50, MX51, MX53, MX54, MX55, MX56, MX57, MX58, MX59, MX6, MX60, MX61, MX62, MX63, MX66, MX67, MX68, MX69, MX7, MX70, MX71, MX72, MX73, MX74, MX75, MX77, MX78, MX8, MX87, MX88, MX89, MX9: footprint SW-MX:SW-Kailh-Hotswap-MX-1.00u -> switch_soldermask:MX100
- MX31: footprint SW-MX:SW-Kailh-Hotswap-MX-2.00u -> switch_soldermask:MX200
- MX35, MX48: footprint SW-MX:SW-Kailh-Hotswap-MX-1.50u -> switch_soldermask:MX150
- MX52, MX76: footprint SW-MX:SW-Kailh-Hotswap-MX-1.75u -> switch_soldermask:MX175
- MX64, MX65: footprint SW-MX:SW-Kailh-Hotswap-MX-2.25u -> switch_soldermask:MX225
- MX79, MX80, MX81, MX83, MX84, MX85, MX86: footprint SW-MX:SW-Kailh-Hotswap-MX-1.25u -> switch_soldermask:MX125
- MX82: footprint SW-MX:SW-Kailh-Hotswap-MX-6.25u -> switch_soldermask:MX625
Other:
- title: Switch Matrix -> mech-eighty schematic
